File: schematic/fault_injection_tool.kicad_pcb (KiCad board)
At the start: 2 copper layers, 53.5 x 66 mm, 7 parts, among them J1 Conn_01x02_Pin, J2 Conn_01x02_Pin, Q1 2N7000

Commit message: Updated schematic drawing and PCB design
Parts:
- R1, R2: footprint Resistor_SMD:R_0201_0603Metric_Pad0.64x0.40mm_HandSolder -> Resistor_SMD:R_0603_1608Metric_Pad0.98x0.95mm_HandSolder
- moved R1 0.06 mm to (122.4, 111.6)
- moved R2 0.06 mm to (120.0, 111.6)
Connections:
- A1 pad 15: unconnected-(A1-MISO-Pad15) -> /lock_state
- A2 pad 16: unconnected-(A2-D1/TX-Pad16) -> /uart_rx
- A2 pad 17: unconnected-(A2-D2-Pad17) -> /uart_tx
Routing:
- net /CTRL: track 63.3 -> 64.8 mm

Commit message: Made some changes to the schematic
Parts:
- added J3: Conn_01x10_Pin, Connector_PinHeader_2.54mm:PinHeader_1x10_P2.54mm_Vertical, F.Cu at (126.3, 78.8)
- moved R1 2.45 mm to (122.8, 114.0), turned to -90 degrees
- moved R2 2.44 mm to (120.4, 114.0), turned to 90 degrees
- moved J1 1.75 mm to (120.2, 103.9)
- moved Q1 0.75 mm to (127.9, 112.1)
Connections:
- net /CTRL renamed /ctrl
- A1 pad 14: unconnected-(A1-MOSI-Pad14) -> /borf
Routing:
- net /uart_rx: track 0.00 -> 62.3 mm
- net /uart_tx: track 0.00 -> 58.7 mm
- net /arduino_gnd: track 30.7 -> 76.1 mm
- net /ctrl: track 64.8 -> 106.0 mm
- net GND: track 39.3 -> 0.00 mm, vias 0 -> 4
- net +5V: track 17.8 -> 47.4 mm
- net /borf: track 0.00 -> 22.3 mm
- net /lock_state: track 0.00 -> 18.7 mm
- added copper zone on B.Cu, net GND
- added copper zone on F.Cu, net GND

Commit message: Updated schematic and pcb layout
Connections:
- A1 pad 14: /borf -> unconnected-(A1-MOSI-Pad14)
- J3 pad 4: /borf -> unconnected-(J3-Pin_4-Pad4)
Routing:
- net /borf: track 22.3 -> 0.00 mm
- net GND: vias 4 -> 33
