File: schematic/fault_injection_tool.kicad_sch (KiCad schematic)
At the start: 7 parts, among them J1 Conn_01x02_Pin, J2 Conn_01x02_Pin, Q1 2N7000

Commit message: Updated schematic drawing and PCB design
Parts:
- added J3: Conn_01x10_Pin, symbol Connector:Conn_01x10_Pin
- R1, R2: footprint Resistor_SMD:R_0201_0603Metric_Pad0.64x0.40mm_HandSolder -> Resistor_SMD:R_0603_1608Metric_Pad0.98x0.95mm_HandSolder
Connections:
- net +5V: now also J3.1 (Pin_1), J3.2 (Pin_2)
- net GND: now also J3.10 (Pin_10), J3.9 (Pin_9)
- net arduino_gnd: now also J3.3 (Pin_3)
- net uart_rx: now reaches A2.16 (D1/TX)
- net uart_tx: now reaches A2.17 (D2)
- net lock_state: now reaches A1.15 (MISO)
Other:
- note added: "Analog Discovery Connection points"
- moved on the sheet: A2, J1, J2, Q1, R1, R2

Commit message: Made some changes to the schematic
Parts:
- J3: footprint (none) -> Connector_PinHeader_2.54mm:PinHeader_1x10_P2.54mm_Vertical
Connections:
- net CTRL is gone; now on net ctrl: A2.15 (D0/RX), J1.1 (Pin_1), R2.1
- net lock_state: now also J3.5 (Pin_5)
- net uart_rx: now also J3.7 (Pin_7)
- net uart_tx: now also J3.8 (Pin_8)
- net borf: now reaches A1.14 (MOSI)
- net borf: now also J3.4 (Pin_4)
- net ctrl: now reaches J3.6 (Pin_6)
Changed lines of the file:
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@@
+	(wire
+		(pts
+			(xy 195.58 53.34) (xy 198.12 53.34)
+		)
+		(stroke
+			(width 0)
+			(type default)
+		)
+	)
+	(wire
+		(pts
+			(xy 41.91 76.2) (xy 44.45 76.2)
+		)
+		(stroke
+			(width 0)
+			(type default)
+		)
+	)
+	(wire
+		(pts
+			(xy 195.58 48.26) (xy 198.12 48.26)
+		)
+		(stroke
+			(width 0)
+			(type default)
+		)
+	)
 	(wire
 		(pts
@@
 	(wire
 		(pts
+			(xy 195.58 50.8) (xy 198.12 50.8)
+		)
+		(stroke
+			(width 0)
+			(type default)
+		)
+	)
+	(wire
+		(pts
 			(xy 90.17 132.08) (xy 90.17 144.78)
 		)
@@
 	(wire
 		(pts
+			(xy 195.58 55.88) (xy 198.12 55.88)
+		)
+		(stroke
+			(width 0)
+			(type default)
+		)
+	)
+	(wire
+		(pts
 			(xy 41.91 78.74) (xy 44.45 78.74)
+		)
+		(stroke
+			(width 0)
+			(type default)
+		)
+	)
+	(wire
+		(pts
+			(xy 195.58 45.72) (xy 198.12 45.72)
 		)
 		(stroke
@@
 		)
 	)
+	(label "uart_rx"
+		(at 198.12 53.34 0)
+		(effects
+			(font
+				(size 1.27 1.27)
+			)
+			(justify left bottom)
+		)
+	)
 	(label "arduino_gnd"
 		(at 198.12 43.18 0)
@@
 		)
 	)
+	(label "uart_tx"
+		(at 198.12 55.88 0)
+		(effects
+			(font
+				(size 1.27 1.27)
+			)
+			(justify left bottom)
+		)
+	)
 	(label "arduino_gnd"
 		(at 93.98 119.38 0)
@@
 		)
 	)
-	(label "CTRL"
+	(label "borf"
+		(at 198.12 45.72 0)
+		(effects
+			(font
+				(size 1.27 1.27)
+			)
+			(justify left bottom)
+		)
+	)
+	(label "lock_state"
+		(at 198.12 48.26 0)
+		(effects
+			(font
+				(size 1.27 1.27)
+			)
+			(justify left bottom)
+		)
+	)
+	(label "borf"
+		(at 41.91 76.2 180)
+		(effects
+			(font
+				(size 1.27 1.27)
+			)
+			(justify right bottom)
+		)
+	)
+	(label "ctrl"
 		(at 57.15 127 0)
 		(effects
@@
 		)
 	)
-	(label "CTRL"
+	(label "ctrl"
+		(at 198.12 50.8 0)
+		(effects
+			(font
+				(size 1.27 1.27)
+			)
+			(justify left bottom)
+		)
+	)
+	(label "ctrl"
 		(at 118.11 45.72 180)
 		(effects
@@
 			)
 		)
-		(property "Footprint" ""
+		(property "Footprint" "Connector_PinHeader_2.54mm:PinHeader_1x10_P2.54mm_Vertical"
 			(at 190.5 48.26 0)
 			(effects

Commit message: Updated schematic and pcb layout
Connections:
- net borf: no longer names the net of A1.14 (MOSI)
- net borf: no longer J3.4 (Pin_4)
Other:
- note added: "Low-side switch"
- note added: "Power header"
- note removed: "Power"
- note removed: "Power drop"
Changed lines of the file:
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@@
 		)
 	)
-	(text "Power drop"
+	(text "Low-side switch"
 		(exclude_from_sim no)
-		(at 31.75 116.84 0)
-		(effects
-			(font
-				(size 1.27 1.27)
-			)
-		)
-	)
-	(text "Power"
+		(at 34.29 116.84 0)
+		(effects
+			(font
+				(size 1.27 1.27)
+			)
+		)
+	)
+	(text "Power header"
 		(exclude_from_sim no)
-		(at 130.81 116.84 0)
+		(at 134.62 116.84 0)
 		(effects
 			(font
@@
 	(wire
 		(pts
-			(xy 41.91 76.2) (xy 44.45 76.2)
-		)
-		(stroke
-			(width 0)
-			(type default)
-		)
-	)
-	(wire
-		(pts
 			(xy 195.58 48.26) (xy 198.12 48.26)
 		)
@@
 		(pts
 			(xy 41.91 78.74) (xy 44.45 78.74)
-		)
-		(stroke
-			(width 0)
-			(type default)
-		)
-	)
-	(wire
-		(pts
-			(xy 195.58 45.72) (xy 198.12 45.72)
 		)
 		(stroke
@@
 		)
 	)
-	(label "borf"
-		(at 198.12 45.72 0)
-		(effects
-			(font
-				(size 1.27 1.27)
-			)
-			(justify left bottom)
-		)
-	)
 	(label "lock_state"
 		(at 198.12 48.26 0)
@@
 		)
 	)
-	(label "borf"
-		(at 41.91 76.2 180)
-		(effects
-			(font
-				(size 1.27 1.27)
-			)
-			(justify right bottom)
-		)
-	)
